File: hw/pcb/credit-card-clock.kicad_sch (KiCad schematic)
At the start: 17 parts, among them J1 Control, J2 Minutes, J3 Hours, J4 Seconds, Q1 2N7002, SW4 SW_DIP_x04, U5 SNx4AHCT08

Commit message: chore: updated to kicad 10
Parts:
- BT1, BT2: value ~ -> (none)
